Commit message: Topico global con mensaje de estados de cada robot

File: ws2/src/articubot_one/description/gazebo_control.xacro (robot description, xacro)
@@ -12,6 +12,7 @@
       <wheel_separation>0.35</wheel_separation>
       <wheel_diameter>0.1</wheel_diameter>
-      <odometry_frame>odom</odometry_frame>
-      <robot_base_frame>base_link</robot_base_frame>
+      <!-- CORRECCIÓN AQUÍ -->
+      <odometry_frame>${namespace}/odom</odometry_frame>
+      <robot_base_frame>${namespace}/base_link</robot_base_frame>
       <publish_odom>true</publish_odom>
       <publish_odom_tf>true</publish_odom_tf>

File: ws2/src/articubot_one/description/lidar.xacro (robot description, xacro)
@@ -2,11 +2,13 @@
 <robot xmlns:xacro="http://www.ros.org/wiki/xacro">
   <xacro:arg name="namespace" default="robot0"/>
-  <xacro:property name="namespace" value="$(arg namespace)"/>
-  <joint name="laser_joint" type="fixed">
-    <parent link="chassis"/>
-    <child link="laser_frame"/>
+  <xacro:property name="prefix" value="${namespace}/"/>
+  <!-- ================= LASER JOINT ================= -->
+  <joint name="${prefix}laser_joint" type="fixed">
+    <parent link="${prefix}chassis"/>
+    <child link="${prefix}laser_frame"/>
     <origin xyz="0.1 0 0.175" rpy="0 0 0"/>
   </joint>
-  <link name="laser_frame">
+  <!-- ================= LASER LINK ================= -->
+  <link name="${prefix}laser_frame">
     <visual>
       <geometry>
@@ -21,7 +23,8 @@
     </collision>
   </link>
-  <gazebo reference="laser_frame">
-  <material>Gazebo/Red</material>
-    <sensor name="laser_sensor" type="ray">
+  <!-- ================= GAZEBO SENSOR ================= -->
+  <gazebo reference="${prefix}laser_frame">
+    <material>Gazebo/Red</material>
+    <sensor name="laser_sensor_${namespace}" type="ray">
       <always_on>true</always_on>
       <visualize>true</visualize>
@@ -41,11 +44,11 @@
       </ray>
       <plugin name="laser_plugin_${namespace}" filename="libgazebo_ros_ray_sensor.so">
-  <ros>
-    <namespace>${namespace}</namespace>
-    <remapping>~/out:=scan</remapping>
-  </ros>
-  <output_type>sensor_msgs/LaserScan</output_type>
-  <frame_name>laser_frame</frame_name>
-</plugin>
+        <ros>
+          <namespace>${namespace}</namespace>
+          <remapping>~/out:=scan</remapping>
+        </ros>
+        <output_type>sensor_msgs/LaserScan</output_type>
+        <frame_name>${prefix}laser_frame</frame_name>
+      </plugin>
     </sensor>
   </gazebo>

File: ws2/src/articubot_one/description/robot_core.xacro (robot description, xacro)
@@ -1,123 +1,122 @@
 <?xml version="1.0"?>
-<robot xmlns:xacro="http://www.ros.org/wiki/xacro" >
-    <xacro:include filename="inertial_macros.xacro" />
-    <!-- Argumento namespace -->
-    <!-- <xacro:arg name="namespace" default="robot0"/>
-    <xacro:property name="namespace" value="$(arg namespace)"/> -->
-    <!--BASE LINK-->
-    <link name="base_link">    </link>
-     <!-- BASE_FOOTPRINT LINK -->
-    <joint name="base_footprint_joint" type="fixed">
-        <parent link="base_link"/>
-        <child link="base_footprint"/>
-        <origin xyz="0 0 0" rpy="0 0 0"/>
-    </joint>
-    <link name="base_footprint">
-    </link>
-    <joint name="chassis_joint" type="fixed">
-        <parent link="base_link"/>
-        <child link="chassis"/>
-        <origin xyz="-0.1 0 0"/>
-    </joint>
-    <!--CHASSIS LINK-->
-    <link name="chassis">
-        <visual>
-            <origin xyz="0.15 0 0.075" rpy="0 0 0"/>
-            <geometry>
-                <box size="0.3 0.3 0.15"/>
-            </geometry>
-            <material name="white"/>
-        </visual>
-        <collision>
-            <origin xyz="0.15 0 0.075" rpy="0 0 0"/>
-            <geometry>
-                <box size="0.3 0.3 0.15"/>
-            </geometry>
-        </collision>
-        <xacro:inertial_box mass="0.5" x="0.3" y="0.3" z="0.15">
-            <origin xyz="0.15 0 0.075" rpy="0 0 0"/>
-        </xacro:inertial_box>
-    </link>
-    <gazebo reference="chassis">
-        <material>Gazebo/White</material>
-    </gazebo>
-    <!-- LEFT WHEEL -->
-    <joint name="left_wheel_joint" type="continuous">
-        <parent link="base_link"/>
-        <child link="left_wheel"/>
-        <origin xyz="0 0.175 0" rpy="-${pi/2} 0 0"/>
-        <axis xyz="0 0 1"/>
-    </joint>
-    <link name="left_wheel">
-        <visual>
-            <geometry>
-                <cylinder length="0.04" radius="0.05" />
-            </geometry>
-            <material name="blue"/>
-        </visual>
-        <collision>
-            <geometry>
-                <cylinder length="0.04" radius="0.05" />
-            </geometry>
-        </collision>
-        <xacro:inertial_cylinder mass="0.1" length="0.05" radius="0.05">
-            <origin xyz="0 0 0" rpy="0 0 0"/>
-        </xacro:inertial_cylinder>
-    </link>
-    <gazebo reference="left_wheel">
-        <material>Gazebo/Blue</material>
-    </gazebo>
-    <!-- RIGHT WHEEL -->
-    <joint name="right_wheel_joint" type="continuous">
-        <parent link="base_link"/>
-        <child link="right_wheel"/>
-        <origin xyz="0 -0.175 0" rpy="${pi/2} 0 0"/>
-        <axis xyz="0 0 -1"/>
-    </joint>
-    <link name="right_wheel">
-        <visual>
-            <geometry>
-                <cylinder length="0.04" radius="0.05" />
-            </geometry>
-            <material name="blue"/>
-        </visual>
-        <collision>
-            <geometry>
-                <cylinder length="0.04" radius="0.05" />
-            </geometry>
-        </collision>
-        <xacro:inertial_cylinder mass="0.1" length="0.05" radius="0.05">
-            <origin xyz="0 0 0" rpy="0 0 0"/>
-        </xacro:inertial_cylinder>
-    </link>
-    <gazebo reference="right_wheel">
-        <material>Gazebo/Blue</material>
-    </gazebo>
-    <!-- CASTER WHEEL -->
-    <joint name="caster_wheel_joint" type="fixed">
-        <parent link="chassis"/>
-        <child link="caster_wheel"/>
-        <origin xyz="0.24 0 0" rpy="0 0 0"/>
-    </joint>
-    <link name="caster_wheel">
-        <visual>
-            <geometry>
-                <sphere radius="0.05" />
-            </geometry>
-            <material name="black"/>
-        </visual>
-        <collision>
-            <geometry>
-                <sphere radius="0.05" />
-            </geometry>
-        </collision>
-        <xacro:inertial_sphere mass="0.1" radius="0.05">
-            <origin xyz="0 0 0" rpy="0 0 0"/>
-        </xacro:inertial_sphere>
-    </link>
-    <gazebo reference="caster_wheel">
-        <material>Gazebo/Black</material>
-        <mu1 value="0.001"/>
-        <mu2 value="0.001"/>
-    </gazebo>
+<robot xmlns:xacro="http://www.ros.org/wiki/xacro">
+  <xacro:include filename="inertial_macros.xacro" />
+  <!-- Namespace argument -->
+  <xacro:arg name="namespace" default="robot0"/>
+  <xacro:property name="prefix" value="${namespace}/"/>
+  <!-- ================= BASE LINK ================= -->
+  <link name="${prefix}base_link"/>
+  <!-- ================= BASE FOOTPRINT ================= -->
+  <joint name="${prefix}base_footprint_joint" type="fixed">
+      <parent link="${prefix}base_link"/>
+      <child link="${prefix}base_footprint"/>
+      <origin xyz="0 0 0" rpy="0 0 0"/>
+  </joint>
+  <link name="${prefix}base_footprint"/>
+  <!-- ================= CHASSIS ================= -->
+  <joint name="${prefix}chassis_joint" type="fixed">
+      <parent link="${prefix}base_link"/>
+      <child link="${prefix}chassis"/>
+      <origin xyz="-0.1 0 0"/>
+  </joint>
+  <link name="${prefix}chassis">
+    <visual>
+        <origin xyz="0.15 0 0.075"/>
+        <geometry>
+            <box size="0.3 0.3 0.15"/>
+        </geometry>
+        <material name="white"/>
+    </visual>
+    <collision>
+        <origin xyz="0.15 0 0.075"/>
+        <geometry>
+            <box size="0.3 0.3 0.15"/>
+        </geometry>
+    </collision>
+    <xacro:inertial_box mass="0.5" x="0.3" y="0.3" z="0.15">
+        <origin xyz="0.15 0 0.075" rpy="0 0 0"/>
+    </xacro:inertial_box>
+</link>
+  <gazebo reference="${prefix}chassis">
+      <material>Gazebo/White</material>
+  </gazebo>
+  <!-- ================= LEFT WHEEL ================= -->
+  <joint name="${prefix}left_wheel_joint" type="continuous">
+      <parent link="${prefix}base_link"/>
+      <child link="${prefix}left_wheel"/>
+      <origin xyz="0 0.175 0" rpy="-${pi/2} 0 0"/>
+      <axis xyz="0 0 1"/>
+  </joint>
+  <link name="${prefix}left_wheel">
+      <visual>
+          <geometry>
+              <cylinder length="0.04" radius="0.05"/>
+          </geometry>
+          <material name="blue"/>
+      </visual>
+      <collision>
+          <geometry>
+              <cylinder length="0.04" radius="0.05"/>
+          </geometry>
+      </collision>
+      <xacro:inertial_cylinder mass="0.1" length="0.05" radius="0.05">
+  <origin xyz="0 0 0" rpy="0 0 0"/>
+</xacro:inertial_cylinder>
+  </link>
+  <gazebo reference="${prefix}left_wheel">
+      <material>Gazebo/Blue</material>
+  </gazebo>
+  <!-- ================= RIGHT WHEEL ================= -->
+  <joint name="${prefix}right_wheel_joint" type="continuous">
+      <parent link="${prefix}base_link"/>
+      <child link="${prefix}right_wheel"/>
+      <origin xyz="0 -0.175 0" rpy="${pi/2} 0 0"/>
+      <axis xyz="0 0 -1"/>
+  </joint>
+  <link name="${prefix}right_wheel">
+      <visual>
+          <geometry>
+              <cylinder length="0.04" radius="0.05"/>
+          </geometry>
+          <material name="blue"/>
+      </visual>
+      <collision>
+          <geometry>
+              <cylinder length="0.04" radius="0.05"/>
+          </geometry>
+      </collision>
+      <xacro:inertial_cylinder mass="0.1" length="0.05" radius="0.05">
+  <origin xyz="0 0 0" rpy="0 0 0"/>
+</xacro:inertial_cylinder>
+  </link>
+  <gazebo reference="${prefix}right_wheel">
+      <material>Gazebo/Blue</material>
+  </gazebo>
+  <!-- ================= CASTER ================= -->
+  <joint name="${prefix}caster_wheel_joint" type="fixed">
+      <parent link="${prefix}chassis"/>
+      <child link="${prefix}caster_wheel"/>
+      <origin xyz="0.24 0 0"/>
+  </joint>
+  <link name="${prefix}caster_wheel">
+      <visual>
+          <geometry>
+              <sphere radius="0.05"/>
+          </geometry>
+          <material name="black"/>
+      </visual>
+      <collision>
+          <geometry>
+              <sphere radius="0.05"/>
+          </geometry>
+      </collision>
+      <xacro:inertial_sphere mass="0.1" radius="0.05">
+  <origin xyz="0 0 0" rpy="0 0 0"/>
+</xacro:inertial_sphere>
+  </link>
+  <gazebo reference="${prefix}caster_wheel">
+      <material>Gazebo/Black</material>
+      <mu1 value="0.001"/>
+      <mu2 value="0.001"/>
+  </gazebo>
 </robot>
