Commit message: Nodo aire, compatibilidad con consenso no R

File: ws3/install/articubot_one/share/articubot_one/description/lidar.xacro (robot description, xacro)
@@ -7,5 +7,5 @@
         <parent link="${namespace}/chassis"/>
         <child link="${namespace}/laser_frame"/>
-        <origin xyz="0.1 0 0.175" rpy="0 0 0"/>
+        <origin xyz="0.25 0 0.175" rpy="0 0 0"/>
     </joint>
     <link name="${namespace}/laser_frame">
